File: hardware/sht45_breakout.kicad_sch (KiCad schematic)
At the start: 6 parts, among them J1 I2C, U1 SHT45-AD1B-R2

Commit message: Switch passives from 0402 to 0603 for hand assembly
Widen the sensor tongue to 4.4 mm so the 0603 decoupling cap still sits
right below the SHT45 with the SDA/SCL lanes beside it, and restack the
pull-ups in the base. Update LCSC numbers (C14663, C25804) and add a
hand-assembly parts list to the README. DRC and schematic/PCB net
comparison still clean.

Co-Authored-By: Claude Opus 5.5 <noreply@anthropic.com>
Claude-Session: https://claude.ai/code/session_01Cw4qgvdZTYbLFFCGBumb2e
Parts:
- C1: footprint Capacitor_SMD:C_0402_1005Metric -> Capacitor_SMD:C_0603_1608Metric; LCSC C1525 -> C14663; Voltage 16V -> 50V
- R1, R2: footprint Resistor_SMD:R_0402_1005Metric -> Resistor_SMD:R_0603_1608Metric; LCSC C25744 -> C25804
Changed lines of the file:
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@@
     (property "Reference" "R1" (at 104.14 87.63 0) (effects (font (size 1.27 1.27)) (justify left)))
     (property "Value" "10k" (at 104.14 90.17 0) (effects (font (size 1.27 1.27)) (justify left)))
-    (property "Footprint" "Resistor_SMD:R_0402_1005Metric" (at 101.6 88.9 0) (effects (font (size 1.27 1.27)) hide))
+    (property "Footprint" "Resistor_SMD:R_0603_1608Metric" (at 101.6 88.9 0) (effects (font (size 1.27 1.27)) hide))
     (property "Datasheet" "" (at 101.6 88.9 0) (effects (font (size 1.27 1.27)) hide))
-    (property "LCSC" "C25744" (at 101.6 88.9 0) (effects (font (size 1.27 1.27)) hide))
+    (property "LCSC" "C25804" (at 101.6 88.9 0) (effects (font (size 1.27 1.27)) hide))
     (property "Tolerance" "1%" (at 101.6 88.9 0) (effects (font (size 1.27 1.27)) hide))
     (pin "1")
@@
     (property "Reference" "R2" (at 114.3 87.63 0) (effects (font (size 1.27 1.27)) (justify left)))
     (property "Value" "10k" (at 114.3 90.17 0) (effects (font (size 1.27 1.27)) (justify left)))
-    (property "Footprint" "Resistor_SMD:R_0402_1005Metric" (at 111.76 88.9 0) (effects (font (size 1.27 1.27)) hide))
+    (property "Footprint" "Resistor_SMD:R_0603_1608Metric" (at 111.76 88.9 0) (effects (font (size 1.27 1.27)) hide))
     (property "Datasheet" "" (at 111.76 88.9 0) (effects (font (size 1.27 1.27)) hide))
-    (property "LCSC" "C25744" (at 111.76 88.9 0) (effects (font (size 1.27 1.27)) hide))
+    (property "LCSC" "C25804" (at 111.76 88.9 0) (effects (font (size 1.27 1.27)) hide))
     (property "Tolerance" "1%" (at 111.76 88.9 0) (effects (font (size 1.27 1.27)) hide))
     (pin "1")
@@
     (property "Reference" "C1" (at 170.18 87.63 0) (effects (font (size 1.27 1.27)) (justify left)))
     (property "Value" "100nF" (at 170.18 90.17 0) (effects (font (size 1.27 1.27)) (justify left)))
-    (property "Footprint" "Capacitor_SMD:C_0402_1005Metric" (at 167.64 88.9 0) (effects (font (size 1.27 1.27)) hide))
+    (property "Footprint" "Capacitor_SMD:C_0603_1608Metric" (at 167.64 88.9 0) (effects (font (size 1.27 1.27)) hide))
     (property "Datasheet" "" (at 167.64 88.9 0) (effects (font (size 1.27 1.27)) hide))
-    (property "LCSC" "C1525" (at 167.64 88.9 0) (effects (font (size 1.27 1.27)) hide))
-    (property "Voltage" "16V" (at 167.64 88.9 0) (effects (font (size 1.27 1.27)) hide))
+    (property "LCSC" "C14663" (at 167.64 88.9 0) (effects (font (size 1.27 1.27)) hide))
+    (property "Voltage" "50V" (at 167.64 88.9 0) (effects (font (size 1.27 1.27)) hide))
     (property "Dielectric" "X7R" (at 167.64 88.9 0) (effects (font (size 1.27 1.27)) hide))
     (pin "1")

Commit message: Add JST XH connector and M2 mounting holes, enlarge board to 16 x 19.8 mm
J2 (JST XH B4B-XH-A) sits right below the 2.54 mm header with the same
VCC/GND/SCL/SDA order. Two M2 holes live on ears either side of the sensor
tongue, separated from it by 1.2 mm milled slots so the thermal
decoupling is kept. Schematic gains J2 and H1/H2; DRC and schematic/PCB
net comparison still clean.

Co-Authored-By: Claude Opus 5.5 <noreply@anthropic.com>
Claude-Session: https://claude.ai/code/session_01Cw4qgvdZTYbLFFCGBumb2e
Parts:
- added H1, H2: M2, MountingHole:MountingHole_2.2mm_M2, symbol Mechanical:MountingHole
- added J2: XH, Connector_JST:JST_XH_B4B-XH-A_1x04_P2.50mm_Vertical, symbol Connector_Generic:Conn_01x04
Connections:
- net GND: now also J2.2 (Pin_2)
- net SCL: now also J2.3 (Pin_3)
- net SDA: now also J2.4 (Pin_4)
- net VCC: now also J2.1 (Pin_1)
Other:
- note added: "J1 (2.54 mm header) / J2 (JST XH 2.50 mm): 1=VCC 2=GND 3=SCL 4=SDA VCC = 1.08 ... 3.6 V (NOT 5 V tolerant!) I2C address 0x44 (SHT45-AD1B), up to 1 MHz (Fm+)"
- note removed: "J1 pinout: 1=VCC 2=GND 3=SCL 4=SDA VCC = 1.08 ... 3.6 V (NOT 5 V tolerant!) I2C address 0x44 (SHT45-AD1B), up to 1 MHz (Fm+)"
Changed lines of the file:
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@@
     (rev "1.0")
     (comment 1 "Sensirion SHT45 humidity & temperature sensor, I2C")
-    (comment 2 "Board 10.2 x 12.5 mm, 2 layers")
+    (comment 2 "Board 16.0 x 19.8 mm, 2 layers, 2x M2 holes")
   )
   (symbol (lib_id "Connector_Generic:Conn_01x04") (at 63.5 88.9 0) (mirror y) (unit 1)
@@
     (effects (font (size 1.27 1.27)) (justify left bottom))
 )
+  (symbol (lib_id "Connector_Generic:Conn_01x04") (at 63.5 66.04 0) (mirror y) (unit 1)
+    (in_bom yes) (on_board yes) (dnp no)
+    (property "Reference" "J2" (at 62.23 60.96 0) (effects (font (size 1.27 1.27)) (justify left)))
+    (property "Value" "XH" (at 62.23 74.93 0) (effects (font (size 1.27 1.27)) (justify left)))
+    (property "Footprint" "Connector_JST:JST_XH_B4B-XH-A_1x04_P2.50mm_Vertical" (at 63.5 66.04 0) (effects (font (size 1.27 1.27)) hide))
+    (property "Datasheet" "" (at 63.5 66.04 0) (effects (font (size 1.27 1.27)) hide))
+    (pin "1")
+    (pin "2")
+    (pin "3")
+    (pin "4")
+    (instances (project "sht45_breakout" (path "/07f6b962-4ebe-5600-9067-22f7fb59b18a" (reference "J2") (unit 1))))
+  )
+  (wire (pts (xy 68.58 63.5) (xy 73.66 63.5)) (stroke (width 0) (type default)))
+  (wire (pts (xy 73.66 63.5) (xy 73.66 58.42)) (stroke (width 0) (type default)))
+  (symbol (lib_id "power:VCC") (at 73.66 58.42 0) (unit 1)
+    (in_bom yes) (on_board yes) (dnp no)
+    (property "Reference" "#PWR005" (at 73.66 52.07 0) (effects (font (size 1.27 1.27)) (justify left) hide))
+    (property "Value" "VCC" (at 72.16 54.42 0) (effects (font (size 1.27 1.27)) (justify left)))
+    (property "Footprint" "" (at 73.66 58.42 0) (effects (font (size 1.27 1.27)) hide))
+    (property "Datasheet" "" (at 73.66 58.42 0) (effects (font (size 1.27 1.27)) hide))
+    (pin "1")
+    (instances (project "sht45_breakout" (path "/07f6b962-4ebe-5600-9067-22f7fb59b18a" (reference "#PWR005") (unit 1))))
+  )
+  (wire (pts (xy 68.58 66.04) (xy 83.82 66.04)) (stroke (width 0) (type default)))
+  (wire (pts (xy 83.82 66.04) (xy 83.82 78.74)) (stroke (width 0) (type default)))
+  (symbol (lib_id "power:GND") (at 83.82 78.74 0) (unit 1)
+    (in_bom yes) (on_board yes) (dnp no)
+    (property "Reference" "#PWR006" (at 83.82 85.09 0) (effects (font (size 1.27 1.27)) (justify left) hide))
+    (property "Value" "GND" (at 82.02 82.94 0) (effects (font (size 1.27 1.27)) (justify left)))
+    (property "Footprint" "" (at 83.82 78.74 0) (effects (font (size 1.27 1.27)) hide))
+    (property "Datasheet" "" (at 83.82 78.74 0) (effects (font (size 1.27 1.27)) hide))
+    (pin "1")
+    (instances (project "sht45_breakout" (path "/07f6b962-4ebe-5600-9067-22f7fb59b18a" (reference "#PWR006") (unit 1))))
+  )
+  (wire (pts (xy 68.58 68.58) (xy 71.12 68.58)) (stroke (width 0) (type default)))
+  (label "SCL" (at 71.12 68.58 0) (fields_autoplaced)
+    (effects (font (size 1.27 1.27)) (justify left bottom))
+)
+  (wire (pts (xy 68.58 71.12) (xy 71.12 71.12)) (stroke (width 0) (type default)))
+  (label "SDA" (at 71.12 71.12 0) (fields_autoplaced)
+    (effects (font (size 1.27 1.27)) (justify left bottom))
+)
+  (symbol (lib_id "Mechanical:MountingHole") (at 190.5 63.5 0) (unit 1)
+    (in_bom no) (on_board yes) (dnp no)
+    (property "Reference" "H1" (at 193.04 62.23 0) (effects (font (size 1.27 1.27)) (justify left)))
+    (property "Value" "M2" (at 193.04 64.77 0) (effects (font (size 1.27 1.27)) (justify left)))
+    (property "Footprint" "MountingHole:MountingHole_2.2mm_M2" (at 190.5 63.5 0) (effects (font (size 1.27 1.27)) hide))
+    (property "Datasheet" "" (at 190.5 63.5 0) (effects (font (size 1.27 1.27)) hide))
+    (instances (project "sht45_breakout" (path "/07f6b962-4ebe-5600-9067-22f7fb59b18a" (reference "H1") (unit 1))))
+  )
+  (symbol (lib_id "Mechanical:MountingHole") (at 203.2 63.5 0) (unit 1)
+    (in_bom no) (on_board yes) (dnp no)
+    (property "Reference" "H2" (at 205.74 62.23 0) (effects (font (size 1.27 1.27)) (justify left)))
+    (property "Value" "M2" (at 205.74 64.77 0) (effects (font (size 1.27 1.27)) (justify left)))
+    (property "Footprint" "MountingHole:MountingHole_2.2mm_M2" (at 203.2 63.5 0) (effects (font (size 1.27 1.27)) hide))
+    (property "Datasheet" "" (at 203.2 63.5 0) (effects (font (size 1.27 1.27)) hide))
+    (instances (project "sht45_breakout" (path "/07f6b962-4ebe-5600-9067-22f7fb59b18a" (reference "H2") (unit 1))))
+  )
   (symbol (lib_id "Device:R") (at 101.6 88.9 0) (unit 1)
     (in_bom yes) (on_board yes) (dnp no)
@@
   (symbol (lib_id "power:VCC") (at 100.33 73.66 0) (unit 1)
     (in_bom yes) (on_board yes) (dnp no)
-    (property "Reference" "#PWR005" (at 100.33 67.31 0) (effects (font (size 1.27 1.27)) (justify left) hide))
+    (property "Reference" "#PWR007" (at 100.33 67.31 0) (effects (font (size 1.27 1.27)) (justify left) hide))
     (property "Value" "VCC" (at 98.83 69.66 0) (effects (font (size 1.27 1.27)) (justify left)))
     (property "Footprint" "" (at 100.33 73.66 0) (effects (font (size 1.27 1.27)) hide))
     (property "Datasheet" "" (at 100.33 73.66 0) (effects (font (size 1.27 1.27)) hide))
     (pin "1")
-    (instances (project "sht45_breakout" (path "/07f6b962-4ebe-5600-9067-22f7fb59b18a" (reference "#PWR005") (unit 1))))
+    (instances (project "sht45_breakout" (path "/07f6b962-4ebe-5600-9067-22f7fb59b18a" (reference "#PWR007") (unit 1))))
   )
   (wire (pts (xy 110.49 73.66) (xy 113.03 73.66)) (stroke (width 0) (type default)))
@@
   (symbol (lib_id "power:VCC") (at 147.32 78.74 0) (unit 1)
     (in_bom yes) (on_board yes) (dnp no)
-    (property "Reference" "#PWR006" (at 147.32 72.39 0) (effects (font (size 1.27 1.27)) (justify left) hide))
+    (property "Reference" "#PWR008" (at 147.32 72.39 0) (effects (font (size 1.27 1.27)) (justify left) hide))
     (property "Value" "VCC" (at 145.82 74.74 0) (effects (font (size 1.27 1.27)) (justify left)))
     (property "Footprint" "" (at 147.32 78.74 0) (effects (font (size 1.27 1.27)) hide))
     (property "Datasheet" "" (at 147.32 78.74 0) (effects (font (size 1.27 1.27)) hide))
     (pin "1")
-    (instances (project "sht45_breakout" (path "/07f6b962-4ebe-5600-9067-22f7fb59b18a" (reference "#PWR006") (unit 1))))
+    (instances (project "sht45_breakout" (path "/07f6b962-4ebe-5600-9067-22f7fb59b18a" (reference "#PWR008") (unit 1))))
   )
   (wire (pts (xy 147.32 96.52) (xy 147.32 99.06)) (stroke (width 0) (type default)))
   (symbol (lib_id "power:GND") (at 147.32 99.06 0) (unit 1)
     (in_bom yes) (on_board yes) (dnp no)
-    (property "Reference" "#PWR007" (at 147.32 105.41 0) (effects (font (size 1.27 1.27)) (justify left) hide))
+    (property "Reference" "#PWR009" (at 147.32 105.41 0) (effects (font (size 1.27 1.27)) (justify left) hide))
     (property "Value" "GND" (at 145.52 103.26 0) (effects (font (size 1.27 1.27)) (justify left)))
     (property "Footprint" "" (at 147.32 99.06 0) (effects (font (size 1.27 1.27)) hide))
     (property "Datasheet" "" (at 147.32 99.06 0) (effects (font (size 1.27 1.27)) hide))
     (pin "1")
-    (instances (project "sht45_breakout" (path "/07f6b962-4ebe-5600-9067-22f7fb59b18a" (reference "#PWR007") (unit 1))))
+    (instances (project "sht45_breakout" (path "/07f6b962-4ebe-5600-9067-22f7fb59b18a" (reference "#PWR009") (unit 1))))
   )
   (symbol (lib_id "Device:C") (at 167.64 88.9 0) (unit 1)
@@
   (symbol (lib_id "power:VCC") (at 167.64 82.55 0) (unit 1)
     (in_bom yes) (on_board yes) (dnp no)
-    (property "Reference" "#PWR008" (at 167.64 76.2 0) (effects (font (size 1.27 1.27)) (justify left) hide))
+    (property "Reference" "#PWR010" (at 167.64 76.2 0) (effects (font (size 1.27 1.27)) (justify left) hide))
     (property "Value" "VCC" (at 166.14 78.55 0) (effects (font (size 1.27 1.27)) (justify left)))
     (property "Footprint" "" (at 167.64 82.55 0) (effects (font (size 1.27 1.27)) hide))
     (property "Datasheet" "" (at 167.64 82.55 0) (effects (font (size 1.27 1.27)) hide))
     (pin "1")
-    (instances (project "sht45_breakout" (path "/07f6b962-4ebe-5600-9067-22f7fb59b18a" (reference "#PWR008") (unit 1))))
+    (instances (project "sht45_breakout" (path "/07f6b962-4ebe-5600-9067-22f7fb59b18a" (reference "#PWR010") (unit 1))))
   )
   (wire (pts (xy 167.64 92.71) (xy 167.64 95.25)) (stroke (width 0) (type default)))
   (symbol (lib_id "power:GND") (at 167.64 95.25 0) (unit 1)
     (in_bom yes) (on_board yes) (dnp no)
-    (property "Reference" "#PWR009" (at 167.64 101.6 0) (effects (font (size 1.27 1.27)) (justify left) hide))
+    (property "Reference" "#PWR011" (at 167.64 101.6 0) (effects (font (size 1.27 1.27)) (justify left) hide))
     (property "Value" "GND" (at 165.84 99.45 0) (effects (font (size 1.27 1.27)) (justify left)))
     (property "Footprint" "" (at 167.64 95.25 0) (effects (font (size 1.27 1.27)) hide))
     (property "Datasheet" "" (at 167.64 95.25 0) (effects (font (size 1.27 1.27)) hide))
     (pin "1")
-    (instances (project "sht45_breakout" (path "/07f6b962-4ebe-5600-9067-22f7fb59b18a" (reference "#PWR009") (unit 1))))
+    (instances (project "sht45_breakout" (path "/07f6b962-4ebe-5600-9067-22f7fb59b18a" (reference "#PWR011") (unit 1))))
   )
   (text "SHT45 I2C breakout" (at 50.8 50.8 0)
     (effects (font (size 2.54 2.54)) (justify left top))
 )
-  (text "J1 pinout: 1=VCC  2=GND  3=SCL  4=SDA\nVCC = 1.08 ... 3.6 V  (NOT 5 V tolerant!)\nI2C address 0x44 (SHT45-AD1B), up to 1 MHz (Fm+)" (at 50.8 114.3 0)
+  (text "J1 (2.54 mm header) / J2 (JST XH 2.50 mm): 1=VCC  2=GND  3=SCL  4=SDA\nVCC = 1.08 ... 3.6 V  (NOT 5 V tolerant!)\nI2C address 0x44 (SHT45-AD1B), up to 1 MHz (Fm+)" (at 50.8 114.3 0)
     (effects (font (size 1.27 1.27)) (justify left top))
 )
